File: 12Vconverter.kicad_sch (KiCad schematic)
At the start: 6 parts, among them IC400 TLP185xSE

Commit message: most changes done
Parts:
- renumbered F402 to F403, IC402 to IC403, IC400 to IC404, R413 to R425, R424 to R426, R425 to R427
