File: 5Vconvector.kicad_sch (KiCad schematic)
At the start: 15 parts, among them Q400 AO3400A, Q403 HSBA8119, U403 INA219AIDCNR

Commit message: most changes done
Parts:
- renumbered C434 to C414, F404 to F402, IC406 to IC402, JP1 to JP402, Q400 to Q403, Q403 to Q405, R419 to R417, R429 to R418, R428 to R419, R430 to R420, R420 to R421, R421 to R422, R422 to R423, R423 to R424, U403 to U404
