File: can-transceiver.kicad_sch (KiCad schematic)
At the start: 4 parts, among them U500 TJA1044GTK_3Z

Commit message: most changes done
Connections:
- net +5V renamed +5V_SB
Changed lines of the file:
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@@
 		(on_board yes)
 		(dnp no)
+		(fields_autoplaced yes)
 		(property "Reference" "#PWR0500"
 			(at 138.43 93.98 0)
@@
 			)
 		)
-		(property "Value" "+5V"
-			(at 138.43 86.36 0)
+		(property "Value" "+5V_SB"
+			(at 138.43 85.09 0)
 			(effects
 				(font
@@
 		)
 		(instances
-			(project "base-module"
+			(project "ATX_PSU"
 				(path "/090a8e41-87a8-4fb1-998b-60a2c0dc4cee/0158e235-e8c1-4e7e-a900-a22642d17049"
-					(reference "#PWR0600")
+					(reference "#PWR0538")
 					(unit 1)
 				)
