File: connector.kicad_sch (KiCad schematic)
At the start: 23 parts, among them IC403 ACS71240, IC410 TLP185xSE, J400 XT60-Angled-F, Q401 HSBA8119, Q402 HSBA8119, Q405 MMBT5551, U404 ADS1115IDGS

Commit message: most changes done
Parts:
- renumbered C428 to C407, C418 to C408, C430 to C411, D404 to D403, D403 to D404, IC403 to IC400, IC410 to IC401, Q405 to Q400, R401 to R400, R414 to R401, R415 to R410, R400 to R413, R417 to R414, R410 to R415, U404 to U403
