File: power.kicad_sch (KiCad schematic)
At the start: 16 parts, among them U301 TPS563201DDCR

Commit message: most changes done
Connections:
- net +5V: no longer C309.1, C310.1, C311.2, U301.3 (VIN), U301.5 (EN)
- new net +5V_SB: C309.1, C310.1, C311.2, U301.3 (VIN), U301.5 (EN)
Changed lines of the file:
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@@
 			)
 		)
-		(property "Value" "+5V"
+		(property "Value" "+5V_SB"
 			(at 48.26 105.41 0)
 			(effects
