File: mcu.kicad_sch (KiCad schematic)
At the start: 44 parts, among them Q404 AO3400A, U405 STM32H562VGTx, X300 Q13FC1350000400, Y400 ASE-xxxMHz

Commit message: most changes done
Parts:
- added R447, R448: 10kΩ, PCM_JLCPCB:R_0402, symbol PCM_JLCPCB-Resistors:0402,10kΩ
Connections:
- net +3V3: now also R447.1, R448.1
- net ADS1115/RDY renamed PWR_OK
- net MASTER_ON renamed MCU_ATX_ON
- net PowerButton renamed Power_Button_IN
- new net I2C.SCL: R447.2
- new net I2C.SDA: R448.2
Other:
- note added: "I2C pull-up resistors"

Commit message: routing progress
Connections:
- net I2C.SCL is gone; now on net I2C1.SCL: R447.2
- net I2C.SDA is gone; now on net I2C1.SDA: R448.2
- net Power_Button_IN: no longer names the net of U405.63 (PC6)
- no-connect marks 47 -> 48
