File: ATX_PSU.kicad_pcb (KiCad board)
At the start: 4 copper layers, 100 x 100 mm, 153 parts, among them IC409 TLP185xSE, J200 09031967921, J400 15246040, J401 Conn_01x06_Pin, J402 ATX-24, J800 USB_C_Receptacle_USB2.0_16P, Q404 AO3400A, Q410 HSBA8119, Q417 HSBA8119, Q700 MMST3904, U100 W25Q128, U301 TPS563201DDCR, U302 CH334P, U400 INA219AIDCNR, U401 TPD2E2U06DCK, U402 TPD2E2U06DCK, U405 STM32H562VGTx, U407 INA219AIDCNR, U408 INA219AIDCNR, U500 TJA1044GTK_3Z, U600 TJA1044GTK_3Z, U700 STM32F103CBTx, U801 FSUSB42UMX, X300 Q13FC1350000400, Y400 ASE-xxxMHz, Y700 8 MHz, Y900 12Mhz

Commit message: removed 3V3 converter
Parts:
- removed C306, C311: 100nF, PCM_JLCPCB:C_0402
- removed C307, C308: 22uF, PCM_JLCPCB:C_0603
- removed C309, C310: 10uF, PCM_JLCPCB:C_0603
- removed D401, D402: Green, PCM_JLCPCB:D_0603
- removed IC409: TLP185xSE, Package_SO:SOIC-4_4.55x3.7mm_P2.54mm
- removed JP301: Test Buck Vout, Jumper:SolderJumper-2_P1.3mm_Open_TrianglePad1.0x1.5mm
- removed L301: 3.3uH, Inductor_SMD:L_Changjiang_FXL0420
- removed R306: 33k2, PCM_JLCPCB:R_0402
- removed R307: 10kΩ, PCM_JLCPCB:R_0402
- removed R411: 470Ω, PCM_JLCPCB:R_0402
- removed R412: 220Ω, PCM_JLCPCB:R_0402
- removed TP302: TestPoint, TestPoint:TestPoint_Pad_D1.0mm
- removed U301: TPS563201DDCR, Package_TO_SOT_SMD:SOT-23-6
- added C409: 100nF, PCM_JLCPCB:C_0402, F.Cu at (83.9, 117.3)
- added C412: 100nF, PCM_JLCPCB:C_0402, F.Cu at (84.4, 122.3)
- added C413: 100nF, PCM_JLCPCB:C_0402, F.Cu at (84.4, 126.3)
- added D400: Green, PCM_JLCPCB:D_0603, F.Cu at (124.4, 95.5)
- added D405: Green, PCM_JLCPCB:D_0603, F.Cu at (128.4, 95.5)
- added D406: Green, PCM_JLCPCB:D_0603, F.Cu at (126.4, 95.5)
- added D407: Green, PCM_JLCPCB:D_0603, F.Cu at (130.4, 95.5)
- added D409: Green, PCM_JLCPCB:D_0603, F.Cu at (132.4, 95.5)
- added D410: Green, PCM_JLCPCB:D_0603, F.Cu at (126.4, 102.3)
- added D411: Green, PCM_JLCPCB:D_0603, F.Cu at (128.4, 102.3)
- added D412: Green, PCM_JLCPCB:D_0603, F.Cu at (130.4, 102.3)
- added F402: 10A, FuseCustom:Fuse_2410_6125, F.Cu at (47.4, 119.3)
- added JP400: SolderJumper_2_Open, Jumper:SolderJumper-2_P1.3mm_Open_RoundedPad1.0x1.5mm, F.Cu at (-92.7, 57.2)
- added JP401: SolderJumper_2_Open, Jumper:SolderJumper-2_P1.3mm_Open_RoundedPad1.0x1.5mm, F.Cu at (-89.9, 82.5)
- added JP402: Test Buck Vout, Jumper:SolderJumper-2_P1.3mm_Open_TrianglePad1.0x1.5mm, F.Cu at (47.3, 112.7)
- added Q409: AO3400A, PCM_JLCPCB:Q_SOT-23, F.Cu at (-83.5, 79.9)
- added Q415: MMBT5551, PCM_JLCPCB:Q_SOT-23, F.Cu at (-20.9, 77.6)
- added Q416: AO3400A, PCM_JLCPCB:Q_SOT-23, F.Cu at (-83.7, 60.2)
- added R405: 10kΩ, PCM_JLCPCB:R_0402, F.Cu at (124.4, 99.0)
- added R406: 10kΩ, PCM_JLCPCB:R_0402, F.Cu at (128.4, 99.0)
- added R407: 10kΩ, PCM_JLCPCB:R_0402, F.Cu at (126.4, 99.0)
- added R408: 10kΩ, PCM_JLCPCB:R_0402, F.Cu at (130.4, 99.0)
- added R431: 10kΩ, PCM_JLCPCB:R_0402, F.Cu at (132.4, 99.0)
- added R432: 10kΩ, PCM_JLCPCB:R_0402, F.Cu at (126.4, 105.8)
- added R433: 10kΩ, PCM_JLCPCB:R_0402, F.Cu at (128.4, 105.8)
- added R444: 10kΩ, PCM_JLCPCB:R_0402, F.Cu at (130.4, 105.8)
- added R446: 10kΩ, PCM_JLCPCB:R_0402, F.Cu at (-31.6, 72.3)
- added R447: 10kΩ, PCM_JLCPCB:R_0402, F.Cu at (-23.3, 94.4)
- added R448: 10kΩ, PCM_JLCPCB:R_0402, F.Cu at (-23.3, 96.3)
- added R449: R, PCM_JLCPCB:R_0402, F.Cu at (106.8, 102.3)
- added R455: 8mΩ, PCM_JLCPCB:R_0805, F.Cu at (80.2, 117.3)
- added R456: 10kΩ, PCM_JLCPCB:R_0402, F.Cu at (-81.4, 85.3)
- added R457: 10kΩ, PCM_JLCPCB:R_0402, F.Cu at (-81.4, 87.2)
- added R458: 22Ω, PCM_JLCPCB:R_0402, F.Cu at (-81.4, 89.0)
- added R464: R, PCM_JLCPCB:R_0402, F.Cu at (106.8, 103.4)
- added R465: 8mΩ, PCM_JLCPCB:R_0805, F.Cu at (80.2, 122.3)
- added R467: 8mΩ, PCM_JLCPCB:R_0805, F.Cu at (80.2, 126.3)
- added R468: 10kΩ, PCM_JLCPCB:R_0402, F.Cu at (-100.0, 57.4)
- added R469: 10kΩ, PCM_JLCPCB:R_0402, F.Cu at (-100.0, 59.2)
- added R470: 22Ω, PCM_JLCPCB:R_0402, F.Cu at (-100.0, 61.1)
- added TP400: TestPoint, TestPoint:TestPoint_Pad_D1.0mm, F.Cu at (151.4, 106.3)
- moved F405 129.1 mm to (66.4, 118.3), turned to 90 degrees
- moved F401 123.5 mm to (60.5, 118.3), turned to 90 degrees
- moved F400 118.0 mm to (54.4, 118.3), turned to 90 degrees
- moved U400 109.0 mm to (75.4, 117.3)
- moved U407 109.0 mm to (75.4, 121.9)
- moved U408 109.0 mm to (75.4, 126.5)
- moved IC408 65.8 mm to (42.4, 83.3), turned to 0 degrees
- moved Q417 61.3 mm to (-92.4, 64.2)
- moved Q410 38.8 mm to (-88.9, 88.2)
- moved REF** 37.7 mm to (108.4, 130.3)
- moved R445 20.2 mm to (106.9, 100.3), turned to 0 degrees
- moved kibuzzard-67B37005 18.8 mm to (151.4, 101.3)
- moved R416 18.4 mm to (118.4, 100.3), turned to 0 degrees
- moved kibuzzard-67E7D86B 16.7 mm to (143.4, 102.3)
- moved kibuzzard-67B37472 16.7 mm to (147.4, 102.3)
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Connections:
- net /ATX connector/PS_ON# renamed /ATX connector/PS_ON#_ATX
- net /ATX connector/PWR_OK renamed /ATX connector/PWR_OK_ATX
- F400 pad 2: unconnected-(F400-Pad2) -> /ATX connector/+3.3V_ATX
- F401 pad 2: +5V -> /ATX connector/+5V_ATX
- F405 pad 2: +12V -> /ATX connector/+12V_ATX
- J400 pad 3: +12V -> /ATX connector/+12V_ATX
- J400 pad 4: +12V -> /ATX connector/+12V_ATX
- J402 pad 1: /ATX connector/+3.3V -> /ATX connector/+3.3V_ATX
- J402 pad 10: +12V -> /ATX connector/+12V_ATX
- J402 pad 11: +12V -> /ATX connector/+12V_ATX
- J402 pad 12: /ATX connector/+3.3V -> /ATX connector/+3.3V_ATX
- J402 pad 13: /ATX connector/+3.3V -> /ATX connector/+3.3V_ATX
- J402 pad 14: /ATX connector/-12V -> /ATX connector/-12V_ATX
- J402 pad 2: /ATX connector/+3.3V -> /ATX connector/+3.3V_ATX
- J402 pad 21: +5V -> /ATX connector/+5V_ATX
- J402 pad 22: +5V -> /ATX connector/+5V_ATX
- J402 pad 23: +5V -> /ATX connector/+5V_ATX
- J402 pad 4: +5V -> /ATX connector/+5V_ATX
- J402 pad 6: +5V -> /ATX connector/+5V_ATX
Routing:
- net /MCU/SWD.~{RST}: track 26.9 -> 127.8 mm
- net /MCU/Buzzer: track 59.6 -> 1.18 mm, vias 2 -> 0
- net +5V: track 40.2 -> 5.43 mm, vias 51 -> 25
- net Net-(BZ401--): track 16.6 -> 5.25 mm
- net Net-(D402-Pad1): track 7.31 -> 0.00 mm
- net Net-(D401-Pad1): track 4.59 -> 0.00 mm
- net /Power/SW_3V3: track 3.24 -> 0.00 mm
- net /Power/+3V3_UNPROTEC: track 3.05 -> 0.00 mm
- net +5V_SB: track 6.73 -> 3.82 mm
- net Net-(Q404-G): track 4.99 -> 2.16 mm
- net /Power/FB_3V3: track 2.43 -> 0.00 mm
- net +3V3: track 57.5 -> 55.1 mm, vias 36 -> 26
- net Net-(D409-Pad2): track 0.00 -> 2.21 mm
- net Net-(D407-Pad1): track 0.00 -> 2.21 mm
- net Net-(D406-Pad1): track 0.00 -> 2.21 mm
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- added copper zone on B.Cu, net +24V
- removed copper zone on F.Cu, net +3V3
- removed copper zone on F.Cu, net /Power/+3V3_UNPROTEC
- removed copper zone on F.Cu, net /Power/SW_3V3
- removed copper zone on F.Cu, net GND

Commit message: routing progress
Parts:
- J402: footprint Connector_Molex:Molex_Mini-Fit_Jr_5569-24A2_2x12_P4.20mm_Horizontal -> Connector_Molex:Molex_Mini-Fit_Jr_5566-24A2_2x12_P4.20mm_Vertical
- moved JP400 175.1 mm to (62.9, 137.4), turned to -90 degrees
- moved R470 171.1 mm to (54.4, 134.8), turned to 90 degrees
- moved R469 171.0 mm to (53.4, 134.8), turned to -90 degrees
- moved R468 169.2 mm to (48.9, 137.8), turned to -90 degrees
- moved Q417 166.9 mm to (58.4, 135.8), turned to -90 degrees
- moved Q416 156.1 mm to (51.8, 137.7)
- moved Q410 137.3 mm to (48.2, 94.6), turned to 90 degrees
- moved JP401 134.1 mm to (43.9, 91.8), turned to 90 degrees
- moved Q409 130.6 mm to (42.9, 112.8), turned to 90 degrees
- moved R456 127.9 mm to (42.9, 115.8)
- moved R458 127.7 mm to (44.6, 109.4), turned to 90 degrees
- moved R457 126.1 mm to (42.8, 109.4), turned to -90 degrees
- moved R447 124.9 mm to (95.4, 133.3), turned to -90 degrees
- moved R448 123.4 mm to (94.4, 133.3), turned to -90 degrees
- moved R446 117.8 mm to (84.9, 54.8), turned to 90 degrees
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Connections:
- net Net-(JP402-B) renamed /ATX connector/3V3_BF
- Q417 pad 1: +12V -> /Power_switch/+12V_sensed
- Q417 pad 2: +12V -> /Power_switch/+12V_sensed
- Q417 pad 3: +12V -> /Power_switch/+12V_sensed
- Q417 pad 5: /Power_switch/+12V_sensed -> +12V
- Q417 pad 6: /Power_switch/+12V_sensed -> +12V
- Q417 pad 7: /Power_switch/+12V_sensed -> +12V
- Q417 pad 8: /Power_switch/+12V_sensed -> +12V
- Q417 pad 9: /Power_switch/+12V_sensed -> +12V
- R447 pad 2: /MCU/I2C.SCL -> /MCU/I2C1.SCL
- R448 pad 2: /MCU/I2C.SDA -> /MCU/I2C1.SDA
- U405 pad 63: /MCU/Power_Button_IN -> unconnected-(U405-PC6-Pad63)
Routing:
- net +5V: track 5.43 -> 219.0 mm, vias 25 -> 61
- net +5V_SB: track 3.82 -> 162.2 mm, vias 0 -> 3
- net /ATX connector/+12V_ATX: track 0.00 -> 145.7 mm, vias 0 -> 15
- net /MCU/I2C1.SCL: track 0.00 -> 126.5 mm, vias 0 -> 4
- net /MCU/I2C1.SDA: track 0.00 -> 125.3 mm, vias 0 -> 4
- net /ATX connector/+5V_ATX: track 0.00 -> 118.7 mm, vias 0 -> 1
- net /MCU/ON-OFF1: track 0.00 -> 106.0 mm, vias 0 -> 2
- net /MCU/ON-OFF0: track 0.00 -> 98.1 mm, vias 0 -> 2
- net +24V: track 0.00 -> 97.1 mm, vias 0 -> 8
- net +12V: track 0.00 -> 91.7 mm, vias 0 -> 4
- net /ATX connector/+3.3V_ATX: track 0.00 -> 87.1 mm
- net /MCU/ON-OFF2: track 0.00 -> 65.6 mm, vias 0 -> 2
- net /ATX connector/PWR_OK_ATX: track 0.00 -> 59.8 mm, vias 0 -> 2
- net /ATX connector/PS_ON#_ATX: track 0.00 -> 42.9 mm, vias 0 -> 2
- net GND: track 83.9 -> 122.6 mm, vias 64 -> 83
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- added copper zone on F.Cu, net +24V
- added copper zone on F.Cu, net /ATX connector/+3.3V_ATX
- added copper zone on F.Cu, net /ATX connector/3V3_BF
- added copper zone on F.Cu, net /Power_switch/+12V_sensed
- added copper zone on F.Cu, net /Power_switch/+5V_sensed

Commit message: finished routing
Parts:
- removed SW400: ~, PS-22F03:SW-TH_G-SWITCH-PS-22F03N
- added SW401: SW_SPDT, Button_Switch_SMD:SW_SPDT_CK_JS102011SAQN, F.Cu at (90.4, 52.8)
- added TP401: TestPoint, TestPoint:TestPoint_Pad_D1.0mm, F.Cu at (127.9, 105.8)
- added TP402: TestPoint, TestPoint:TestPoint_Pad_D1.0mm, F.Cu at (125.9, 105.8)
- JP402: footprint Jumper:SolderJumper-2_P1.3mm_Open_TrianglePad1.0x1.5mm -> Jumper:SolderJumper-2_P1.3mm_Bridged_RoundedPad1.0x1.5mm
- moved REF** 54.2 mm to (104.9, 130.3)
- moved kibuzzard-67B37005 21.6 mm to (129.9, 103.3)
- moved TP400 21.5 mm to (129.9, 105.8)
- moved kibuzzard-67B37472 19.5 mm to (127.9, 103.3)
- moved kibuzzard-67E7D86B 17.5 mm to (125.9, 103.3)
- moved Q415 11.5 mm to (91.4, 60.8), turned to 90 degrees
- moved R446 8.28 mm to (88.4, 62.3)
Routing:
- net /MCU/MCU_ATX_ON: track 0.00 -> 60.8 mm, vias 0 -> 2
- net +5V_SB: track 162.2 -> 215.4 mm
- net /ATX connector/PS_ON#_ATX: track 42.9 -> 57.1 mm
- net GND: track 122.6 -> 132.1 mm, vias 83 -> 85
- net Net-(Q415-B): track 0.00 -> 2.07 mm
- net +3V3: track 75.2 -> 76.7 mm, vias 40 -> 41
