File: backplane.kicad_sch (KiCad schematic)
At the start: 2 parts, among them J200 09031967921, U402 TPD2E2U06DCK

Commit message: most changes done
Connections:
- net +5V_STDBY renamed +5V
Changed lines of the file:
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@@
 			)
 		)
-		(property "Value" "+5V_STDBY"
-			(at 150.622 27.94 90)
+		(property "Value" "+5V"
+			(at 147.066 27.94 90)
 			(effects
 				(font
@@
 			)
 		)
-		(property "Value" "+5V_STDBY"
+		(property "Value" "+5V"
 			(at 269.24 92.71 0)
 			(effects
@@
 			)
 		)
-		(property "Value" "+5V_STDBY"
-			(at 62.738 27.94 90)
+		(property "Value" "+5V"
+			(at 66.04 28.448 90)
 			(effects
 				(font
@@
 			)
 		)
-		(property "Value" "+5V_STDBY"
-			(at 64.008 111.76 90)
-			(effects
-				(font
+		(property "Value" "+5V"
+			(at 67.056 111.76 90)
+			(effects
+				(font

Commit message: finished routing
Parts:
- added TP401, TP402: TestPoint, TestPoint:TestPoint_Pad_D1.0mm, symbol Connector:TestPoint
Connections:
- net GND: now also TP402.1
- new net +5V_SB: TP401.1
